Commit message: after x amount of hours, thins kindof works?

File: catkin_ws/src/pybullet_simulator/robots/ur_description/urdf/ur10_robot.urdf (robot description, URDF)
Before this commit: robot ur10, 11 links, 10 joints
Joints:
- joint world_joint: origin xyz=0.0 0.0 0.0 rpy=0.0 0.0 0.0 -> xyz=0 0 0.5 rpy=0.0 0.0 0.0
