Commit message: working realsense

File: catkin_ws/src/pybullet_simulator/robots/ur_description/urdf/myrg2ur10.urdf (robot description, URDF)
Before this commit: robot rg2myur10, 20 links, 19 joints
Links:
- added link realsense_camera_frame, mass 1e-6
- added link realsense_color_optical_frame, mass 1e-6
- added link realsense_depth_optical_frame
- added link realsense_link, mass 0.072; collision box size=0.02505 0.09 0.025; visual mesh filename=package://realsense2_description/meshes/d435.dae
Joints:
- added joint realsense_camera_joint: type fixed, parent hand_link, child realsense_link, origin xyz=0.05 0 0.028 rpy=0 0 0
- added joint realsense_fake_joint: type fixed, parent realsense_link, child realsense_camera_frame, origin xyz=0.0 0.015 0.0 rpy=0.0 0.0 0.0
- added joint realsense_optical_joint: type fixed, parent realsense_link, child realsense_color_optical_frame, origin xyz=0.0 0.015 0.0 rpy=-1.571 0 -1.571
- added joint realsense_rgb2depth_virtual_joint: type fixed, parent realsense_color_optical_frame, child realsense_depth_optical_frame, origin xyz=0.0 0.0 0.0 rpy=0.0 0.0 0.0
