Commit message: added git ignore

File: catkin_ws/src/myur10_description/urdf/myur10.urdf (robot description, URDF)
Before this commit: robot myur10, 12 links, 11 joints
Links:
- link table: geometry collision mesh filename=package://myur10_description/meshes/table/collision/table.o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; visual mesh filename=package://myur10_description/meshes/table/visual/table.dae

File: catkin_ws/src/myur10_description/urdf/myur10.urdf.xacro (robot description, xacro)
@@ -13,5 +13,5 @@
     <visual>
       <geometry>
-        <mesh filename="$(find myur10_description)/meshes/table/visual/table.dae"/>
+        <mesh filename="package://myur10_description/meshes/table/visual/table.dae"/>
       </geometry>
       <material name="grey"/>
@@ -19,5 +19,5 @@
     <collision>
       <geometry>
-        <mesh filename="$(find myur10_description)/meshes/table/collision/table.obj"/>
+        <mesh filename="package://myur10_description/meshes/table/collision/table.obj"/>
       </geometry>
     </collision>
