Commit message: Solved problems leading to not being able to move the robot

File: catkin_ws/src/myur10_description/urdf/myrg2ur10.urdf.xacro (robot description, xacro)
@@ -31,5 +31,5 @@
       <parent link="tool0"/>
         <child link="rg2_base_link"/>
-      <origin xyz="0 0 0.004" rpy="0 ${-pi/2.0} 0"/>
+      <origin xyz="0 0 0.05" rpy="0 ${-pi/2.0} 0"/>
     </joint>
     <joint name="base_joint" type="fixed">

File: catkin_ws/src/pybullet_simulator/robots/ur_description/urdf/myrg2ur10.urdf (robot description, URDF)
Before this commit: robot rg2myur10, 24 links, 23 joints
Joints:
- joint realsense_camera_joint: origin xyz=0.05 0 0.028 rpy=0 0 0 -> xyz=0.08 0 0.035 rpy=0 0 0
