Commit message: Changed camera position, camera picture positions

File: myur10_description/urdf/myrg2ur10.urdf (robot description, URDF)
Before this commit: robot rg2myur10, 20 links, 19 joints
Joints:
- joint ee_rg2_fixed_joint: origin xyz=0 0 0.004 rpy=0 -1.570796327 0 -> xyz=1 0 0.01 rpy=0 -1.570796327 0

File: pybullet_simulator/robots/ur_description/urdf/myrg2ur10.urdf (robot description, URDF)
Before this commit: robot rg2myur10, 24 links, 23 joints
Joints:
- joint realsense_camera_joint: origin xyz=0.05 0 0.028 rpy=0 0 0 -> xyz=0.1 0 0.038 rpy=0 0 0

Commit message: Took pictures of the simulation, fixed robotgripper angle

File: myur10_description/urdf/myrg2ur10.urdf (robot description, URDF)
Before this commit: robot rg2myur10, 20 links, 19 joints
Links:
- added link gripper_mid
- added link realsense_camera_frame, mass 1e-6
- added link realsense_color_optical_frame, mass 1e-6
- added link realsense_depth_optical_frame
- added link realsense_link, mass 0.072; collision box size=0.02505 0.09 0.025; visual mesh filename=package://realsense2_description/meshes/d435.dae
Joints:
- added joint camera_joint: type fixed, parent hand_link, child realsense_link, origin xyz=0.088 0 0.046  rpy=0 0 0
- added joint gripper_mid_joint: type fixed, parent tool0, child gripper_mid, origin xyz=0 0 0.2 rpy=0 0 0
- added joint realsense_fake_joint: type fixed, parent realsense_link, child realsense_camera_frame, origin xyz=0.0 0.015 0.0 rpy=0.0 0.0 0.0
- added joint realsense_optical_joint: type fixed, parent realsense_link, child realsense_color_optical_frame, origin xyz=0.0 0.015 0.0 rpy=-1.571 0 -1.571
- added joint realsense_rgb2depth_virtual_joint: type fixed, parent realsense_color_optical_frame, child realsense_depth_optical_frame, origin xyz=0.0 0.0 0.0 rpy=0.0 0.0 0.0
- joint base_joint: origin xyz=0 0 0 rpy=0.0 0.0 0.0 -> xyz=0.0 0.0 0.0 rpy=0.0 0.0 0.0
- joint ee_rg2_fixed_joint: origin xyz=1 0 0.01 rpy=0 -1.570796327 0 -> xyz=0 0 0.004 rpy=3.1415 -1.570796327 0
- joint wrist_3_joint: origin xyz=0.0 0.0 0.1157 rpy=0.0 0.0 0.0 -> xyz=0.0 0.0 0.1157 rpy=0.0 1.5707 0.0
- joint wrist_3_link-tool0_fixed_joint: origin xyz=0 0.0922 0 rpy=-1.570796327 0 0 -> xyz=0 0.0922 0 rpy=-1.570796327 -1.570796 0

File: myur10_description/urdf/myrg2ur10.urdf.xacro (robot description, xacro)
@@ -31,10 +31,17 @@
       <parent link="tool0"/>
         <child link="rg2_base_link"/>
-      <origin xyz="0 0 0.004" rpy="0 ${-pi/2.0} 0"/>
+      <origin xyz="0 0 0.004" rpy="${pi} ${-pi/2.0} 0"/>
     </joint>
+    <link name="gripper_mid"/>
+    <joint name="gripper_mid_joint" type="fixed">
+      <parent link="tool0"/>
+        <child link="gripper_mid"/>
+      <origin xyz="0 0 0.2" rpy="0 0 0"/>
+    </joint>
+    <xacro:arg name="use_nominal_extrinsics" default="false" />
     <joint name="base_joint" type="fixed">
       <parent link="world"/>
       <child link="base_link"/>
-      <origin xyz ="0 0 0" rpy="0.0 0.0 0.0"/>
+      <origin xyz ="0.0 0 0.0" rpy="0.0 0.0 0.0"/>
     </joint>
 </robot>

File: pybullet_simulator/robots/ur_description/urdf/myrg2ur10.urdf (robot description, URDF)
Before this commit: robot rg2myur10, 24 links, 23 joints
Links:
- added link gripper_mid
Joints:
- removed joint realsense_camera_joint
- added joint camera_joint: type fixed, parent hand_link, child realsense_link, origin xyz=0.088 0 0.046  rpy=0 0 0
- added joint gripper_mid_joint: type fixed, parent tool0, child gripper_mid, origin xyz=0 0 0.2 rpy=0 0 0
- joint base_joint: origin xyz=0 0 0 rpy=0.0 0.0 0.0 -> xyz=-0.42 0 0.0 rpy=0.0 0.0 0.0
- joint ee_rg2_fixed_joint: origin xyz=0 0 0.004 rpy=0 -1.570796327 0 -> xyz=0 0 0.004 rpy=3.1415 -1.570796327 0
- joint world_link: origin xyz=0.42 0.0 -0.39 rpy=0.0 0.0 0.0 -> xyz=0.0 0.0 -0.39 rpy=0.0 0.0 0.0
- joint wrist_3_joint: origin xyz=0.0 0.0 0.1157 rpy=0.0 0.0 0.0 -> xyz=0.0 0.0 0.1157 rpy=0.0 1.5707 0.0
- joint wrist_3_link-tool0_fixed_joint: origin xyz=0 0.0922 0 rpy=-1.570796327 0 0 -> xyz=0 0.0922 0 rpy=-1.570796327 1.570796 0

File: universal_robot/ur_description/urdf/ur10.urdf.xacro (robot description, xacro)
@@ -269,5 +269,5 @@
       <parent link="${prefix}wrist_2_link" />
       <child link = "${prefix}wrist_3_link" />
-      <origin xyz="0.0 0.0 ${wrist_2_length}" rpy="0.0 0.0 0.0" />
+      <origin xyz="0.0 0.0 ${wrist_2_length}" rpy="0.0 1.5707 0.0" />
       <axis xyz="0 1 0" />
       <xacro:unless value="${joint_limited}">
@@ -332,5 +332,5 @@
     <link name="${prefix}tool0"/>
     <joint name="${prefix}wrist_3_link-tool0_fixed_joint" type="fixed">
-      <origin xyz="0 ${wrist_3_length} 0" rpy="${pi/-2.0} 0 0"/>
+      <origin xyz="0 ${wrist_3_length} 0" rpy="${pi/-2.0} ${pi/2.0} 0"/>
       <parent link="${prefix}wrist_3_link"/>
       <child link="${prefix}tool0"/>
