Commit message: missed files in last commit

File: cobotsA_config/ur10_cobotsA.xacro (robot description, xacro)
@@ -41,5 +41,10 @@
     <origin xyz="0.0 0.0 0.0" rpy="0.0 0.0 1.5707"/>
   </joint>
+  <xacro:arg name="use_nominal_extrinsics" default="false" />
+  <xacro:include filename="$(find realsense2_description)/urdf/_d435.urdf.xacro"/>
   <xacro:include filename="$(find ur_description)/urdf/inc/ur10_macro.xacro"/>
   <xacro:ur10_robot prefix="" />
+  <xacro:sensor_d435 parent="wrist_3_link" use_nominal_extrinsics="$(arg use_nominal_extrinsics)">
+    <origin xyz="0 -0.046 -0.08" rpy="0 -1.5707 1.5707"/>
+  </xacro:sensor_d435>
 </robot>

File: myur10_description/urdf/myrg2ur10.urdf.xacro (robot description, xacro)
@@ -24,8 +24,7 @@
   </link>
     <xacro:arg name = "transmission_hw_interface" default = "hardware_interface/PositionJointInterface"/>
-    <xacro:include filename = "$(find ur_description)/urdf/common.gazebo.xacro"/>
-    <xacro:include filename = "$(find ur_description)/urdf/ur10.urdf.xacro"/>
+    <xacro:include filename = "$(find ur_description)/urdf/ur10.xacro"/>
     <xacro:include filename = "$(find rg2_description)/urdf/rg2.urdf.xacro"/>
-    <xacro:ur10_robot prefix="" joint_limited="true" transmission_hw_interface= "$(arg transmission_hw_interface)"/>
+    <xacro:ur10_robot prefix="" transmission_hw_interface= "$(arg transmission_hw_interface)"/>
     <joint name="ee_rg2_fixed_joint" type="fixed">
       <parent link="tool0"/>

Commit message: all the changes on the borrowed laptop

File: cobotsA_config/ur10_cobotsA.xacro (robot description, xacro)
@@ -44,7 +44,13 @@
   <xacro:include filename="$(find realsense2_description)/urdf/_d435.urdf.xacro"/>
   <xacro:include filename="$(find ur_description)/urdf/inc/ur10_macro.xacro"/>
+  <xacro:include filename="$(find rg2_description)/urdf/rg2.urdf.xacro"/>
+    <joint name ="rg2_fixed_joint" type="fixed">
+    <parent link="tool0"/>
+    <child link="rg2_base_link"/>
+    <origin xyz="0.0 0.0 0.0" rpy="0.0 -1.5707 1.5707"/>
+  </joint>
   <xacro:ur10_robot prefix="" />
-  <xacro:sensor_d435 parent="wrist_3_link" use_nominal_extrinsics="$(arg use_nominal_extrinsics)">
-    <origin xyz="0 -0.046 -0.08" rpy="0 -1.5707 1.5707"/>
+  <xacro:sensor_d435 parent="hand_link" use_nominal_extrinsics="$(arg use_nominal_extrinsics)">
+    <origin xyz="0.088 0.0 0.046" rpy="0 0 0"/>
   </xacro:sensor_d435>
 </robot>
